Commit message: Sucessfully built first differential drive bot

File: first_robot.urdf (robot description, URDF)
Before this commit: robot first_robot, 1 links, 0 joints
Links:
- added link base_footprint
- added link caster_wheel_link; visual sphere radius=0.05
- added link left_wheel_link; visual cylinder length=0.05 radius=0.15
- added link lidar_link; visual cylinder length=0.05 radius=0.1
- added link right_wheel_link; visual cylinder length=0.05 radius=0.15
Joints:
- added joint base_caster_wheel_joint: type fixed, parent base_link, child caster_wheel_link, origin xyz=0.2 0 -0.025 rpy=0 0 0
- added joint base_footprint_joint: type fixed, parent base_footprint, child base_link, origin xyz=0 0 0.05 rpy=0 0 0
- added joint base_left_wheel_joint: type continuous, parent base_link, child left_wheel_link, origin xyz=-0.15 0.225 0.05 rpy=-1.5708 0 0, axis 0 0 1
- added joint base_lidar_joint: type fixed, parent base_link, child lidar_link, origin xyz=0 0 0.225 rpy=0 0 0
- added joint base_right_wheel_joint: type continuous, parent base_link, child right_wheel_link, origin xyz=-0.15 -0.225 0.05 rpy=1.5708 0 0, axis 0 0 1
